File: hardware/mainboard/mainboard.sch (KiCad schematic (older format))
At the start: 19 parts

Commit message: update led resistors
Parts:
- gave numbers to parts that had none: 5
- renumbered BT-LIPO to BT-LIPO1, DBLU to DBLU1, DERR to DERR1, DGRN to DGRN1, DRED to DRED1, DYEL to DYEL1, JDIAG to JDIAG1, SW-BLU to SW-BLU1, SW-GRN to SW-GRN1, SW-PWR to SW-PWR1, SW-RED to SW-RED1, SW-YEL to SW-YEL1
Other:
- moved on the sheet: R2, R3, R4, R5
Changed lines of the file:
@@
 $EndDescr
 $Comp
-L Device:LED DRED
+L Device:LED DRED1
 U 1 1 61BE3269
 P 7250 5550
-F 0 "DRED" H 7242 5295 50  0000 C CNN
+F 0 "DRED1" H 7242 5295 50  0000 C CNN
 F 1 "LED" H 7242 5386 50  0000 C CNN
 F 2 "" H 7250 5550 50  0001 C CNN
@@
 $EndComp
 $Comp
-L Device:LED DYEL
+L Device:LED DYEL1
 U 1 1 61BE3495
 P 7250 5150
-F 0 "DYEL" H 7242 4895 50  0000 C CNN
+F 0 "DYEL1" H 7242 4895 50  0000 C CNN
 F 1 "LED" H 7242 4986 50  0000 C CNN
 F 2 "" H 7250 5150 50  0001 C CNN
@@
 $EndComp
 $Comp
-L Device:LED DBLU
+L Device:LED DBLU1
 U 1 1 61BE399E
 P 7250 4350
-F 0 "DBLU" H 7242 4095 50  0000 C CNN
+F 0 "DBLU1" H 7242 4095 50  0000 C CNN
 F 1 "LED" H 7242 4186 50  0000 C CNN
 F 2 "" H 7250 4350 50  0001 C CNN
@@
 $EndComp
 $Comp
-L Device:LED DGRN
+L Device:LED DGRN1
 U 1 1 61BE39F4
 P 7250 4750
-F 0 "DGRN" H 7242 4495 50  0000 C CNN
+F 0 "DGRN1" H 7242 4495 50  0000 C CNN
 F 1 "LED" H 7242 4586 50  0000 C CNN
 F 2 "" H 7250 4750 50  0001 C CNN
@@
 $EndComp
 $Comp
-L Device:LED DERR
+L Device:LED DERR1
 U 1 1 61BE4930
 P 7250 3950
-F 0 "DERR" H 7242 3695 50  0000 C CNN
+F 0 "DERR1" H 7242 3695 50  0000 C CNN
 F 1 "LED" H 7242 3786 50  0000 C CNN
 F 2 "" H 7250 3950 50  0001 C CNN
@@
 $EndComp
 $Comp
-L Device:R R?
+L Device:R R1
 U 1 1 61BE5850
 P 7700 3950
-F 0 "R?" V 7493 3950 50  0000 C CNN
+F 0 "R1" V 7493 3950 50  0000 C CNN
 F 1 "R" V 7584 3950 50  0000 C CNN
 F 2 "" V 7630 3950 50  0001 C CNN
@@
 $EndComp
 $Comp
-L Device:R R?
+L Device:R R2
 U 1 1 61BE5A1D
-P 7700 4400
-F 0 "R?" V 7493 4400 50  0000 C CNN
-F 1 "R" V 7584 4400 50  0000 C CNN
-F 2 "" V 7630 4400 50  0001 C CNN
-F 3 "~" H 7700 4400 50  0001 C CNN
-	1    7700 4400
-	0    1    1    0
-$EndComp
-$Comp
-L Device:R R?
+P 7700 4350
+F 0 "R2" V 7493 4350 50  0000 C CNN
+F 1 "R" V 7584 4350 50  0000 C CNN
+F 2 "" V 7630 4350 50  0001 C CNN
+F 3 "~" H 7700 4350 50  0001 C CNN
+	1    7700 4350
+	0    1    1    0
+$EndComp
+$Comp
+L Device:R R3
 U 1 1 61BE5A49
-P 7700 4800
-F 0 "R?" V 7493 4800 50  0000 C CNN
-F 1 "R" V 7584 4800 50  0000 C CNN
-F 2 "" V 7630 4800 50  0001 C CNN
-F 3 "~" H 7700 4800 50  0001 C CNN
-	1    7700 4800
-	0    1    1    0
-$EndComp
-$Comp
-L Device:R R?
+P 7700 4750
+F 0 "R3" V 7493 4750 50  0000 C CNN
+F 1 "R" V 7584 4750 50  0000 C CNN
+F 2 "" V 7630 4750 50  0001 C CNN
+F 3 "~" H 7700 4750 50  0001 C CNN
+	1    7700 4750
+	0    1    1    0
+$EndComp
+$Comp
+L Device:R R4
 U 1 1 61BE5A77
-P 7700 5200
-F 0 "R?" V 7493 5200 50  0000 C CNN
-F 1 "R" V 7584 5200 50  0000 C CNN
-F 2 "" V 7630 5200 50  0001 C CNN
-F 3 "~" H 7700 5200 50  0001 C CNN
-	1    7700 5200
-	0    1    1    0
-$EndComp
-$Comp
-L Device:R R?
+P 7700 5150
+F 0 "R4" V 7493 5150 50  0000 C CNN
+F 1 "R" V 7584 5150 50  0000 C CNN
+F 2 "" V 7630 5150 50  0001 C CNN
+F 3 "~" H 7700 5150 50  0001 C CNN
+	1    7700 5150
+	0    1    1    0
+$EndComp
+$Comp
+L Device:R R5
 U 1 1 61BE5AA7
-P 7700 5600
-F 0 "R?" V 7493 5600 50  0000 C CNN
-F 1 "R" V 7584 5600 50  0000 C CNN
-F 2 "" V 7630 5600 50  0001 C CNN
-F 3 "~" H 7700 5600 50  0001 C CNN
-	1    7700 5600
+P 7700 5550
+F 0 "R5" V 7493 5550 50  0000 C CNN
+F 1 "R" V 7584 5550 50  0000 C CNN
+F 2 "" V 7630 5550 50  0001 C CNN
+F 3 "~" H 7700 5550 50  0001 C CNN
+	1    7700 5550
 	0    1    1    0
 $EndComp
@@
 	7400 3950 7550 3950
 Wire Wire Line
-	7400 4350 7550 4400
-Wire Wire Line
-	7400 4750 7550 4800
-Wire Wire Line
-	7400 5150 7550 5200
-Wire Wire Line
-	7400 5550 7550 5600
-$Comp
-L Device:Battery_Cell BT-LIPO
+	7400 4350 7550 4350
+Wire Wire Line
+	7400 4750 7550 4750
+Wire Wire Line
+	7400 5150 7550 5150
+Wire Wire Line
+	7400 5550 7550 5550
+$Comp
+L Device:Battery_Cell BT-LIPO1
 U 1 1 61BE7ABB
 P 5000 5700
-F 0 "BT-LIPO" H 5118 5796 50  0000 L CNN
+F 0 "BT-LIPO1" H 5118 5796 50  0000 L CNN
 F 1 "Battery_Cell" H 5118 5705 50  0000 L CNN
 F 2 "" V 5000 5760 50  0001 C CNN
@@
 	5000 5800 5000 5850
 $Comp
-L Switch:SW_Push SW-RED
+L Switch:SW_Push SW-RED1
 U 1 1 61BF1126
 P 2900 3250
-F 0 "SW-RED" H 2900 3535 50  0000 C CNN
+F 0 "SW-RED1" H 2900 3535 50  0000 C CNN
 F 1 "SW_Push" H 2900 3444 50  0000 C CNN
 F 2 "" H 2900 3450 50  0001 C CNN
@@
 $EndComp
 $Comp
-L Switch:SW_Push SW-YEL
+L Switch:SW_Push SW-YEL1
 U 1 1 61BF11C9
 P 2900 3650
-F 0 "SW-YEL" H 2900 3935 50  0000 C CNN
+F 0 "SW-YEL1" H 2900 3935 50  0000 C CNN
 F 1 "SW_Push" H 2900 3844 50  0000 C CNN
 F 2 "" H 2900 3850 50  0001 C CNN
@@
 $EndComp
 $Comp
-L Switch:SW_Push SW-GRN
+L Switch:SW_Push SW-GRN1
 U 1 1 61BF1205
 P 2900 4050
-F 0 "SW-GRN" H 2900 4335 50  0000 C CNN
+F 0 "SW-GRN1" H 2900 4335 50  0000 C CNN
 F 1 "SW_Push" H 2900 4244 50  0000 C CNN
 F 2 "" H 2900 4250 50  0001 C CNN
@@
 $EndComp
 $Comp
-L Switch:SW_Push SW-BLU
+L Switch:SW_Push SW-BLU1
 U 1 1 61BF1241
 P 2900 4450
-F 0 "SW-BLU" H 2900 4735 50  0000 C CNN
+F 0 "SW-BLU1" H 2900 4735 50  0000 C CNN
 F 1 "SW_Push" H 2900 4644 50  0000 C CNN
 F 2 "" H 2900 4650 50  0001 C CNN
@@
 	1    0    0    -1
 $EndComp
-Wire Wire Line
-	7850 5800 7850 5600
 $Comp
 L MCU_Module_2:Adafruit_Feather_M0_Basic_Proto A1
@@
 	6900 2950 6900 3150
 $Comp
-L power:GND #PWR?
+L power:GND #PWR04
 U 1 1 61BFBBCD
 P 7350 2200
-F 0 "#PWR?" H 7350 1950 50  0001 C CNN
+F 0 "#PWR04" H 7350 1950 50  0001 C CNN
 F 1 "GND" H 7355 2027 50  0000 C CNN
 F 2 "" H 7350 2200 50  0001 C CNN
@@
 	7350 2450 7100 2450
 $Comp
-L power:VCC #PWR?
+L power:VCC #PWR03
 U 1 1 61BFD431
 P 7100 2200
-F 0 "#PWR?" H 7100 2050 50  0001 C CNN
+F 0 "#PWR03" H 7100 2050 50  0001 C CNN
 F 1 "VCC" H 7117 2373 50  0000 C CNN
 F 2 "" H 7100 2200 50  0001 C CNN
@@
 NoConn ~ 7350 2950
 $Comp
-L power:VBUS #PWR?
+L power:VBUS #PWR06
 U 1 1 61C06D81
 P 8900 2200
-F 0 "#PWR?" H 8900 2050 50  0001 C CNN
+F 0 "#PWR06" H 8900 2050 50  0001 C CNN
 F 1 "VBUS" H 8915 2373 50  0000 C CNN
 F 2 "" H 8900 2200 50  0001 C CNN
@@
 	2700 4050 2700 4450
 $Comp
-L power:VBUS #PWR?
+L power:VBUS #PWR01
 U 1 1 61C1FE9A
 P 4250 4900
-F 0 "#PWR?" H 4250 4750 50  0001 C CNN
+F 0 "#PWR01" H 4250 4750 50  0001 C CNN
 F 1 "VBUS" H 4265 5073 50  0000 C CNN
 F 2 "" H 4250 4900 50  0001 C CNN
@@
 Should VIO on the Notecarrier be wired to 3.3V on the Feather?
 $Comp
-L power:+3V3 #PWR?
+L power:+3V3 #PWR02
 U 1 1 61C24AE2
 P 4350 5250
-F 0 "#PWR?" H 4350 5100 50  0001 C CNN
+F 0 "#PWR02" H 4350 5100 50  0001 C CNN
 F 1 "+3V3" H 4365 5423 50  0000 C CNN
 F 2 "" H 4350 5250 50  0001 C CNN
@@
 $EndComp
 $Comp
-L power:+3V3 #PWR?
+L power:+3V3 #PWR05
 U 1 1 61C24B89
 P 8600 2200
-F 0 "#PWR?" H 8600 2050 50  0001 C CNN
+F 0 "#PWR05" H 8600 2050 50  0001 C CNN
 F 1 "+3V3" H 8615 2373 50  0000 C CNN
 F 2 "" H 8600 2200 50  0001 C CNN
@@
 	8600 2350 9150 2350
 $Comp
-L Connector:Conn_01x04_Female JDIAG
+L Connector:Conn_01x04_Female JDIAG1
 U 1 1 61C2E1B9
 P 9500 2650
-F 0 "JDIAG" H 9527 2626 50  0000 L CNN
+F 0 "JDIAG1" H 9527 2626 50  0000 L CNN
 F 1 "Conn_01x04_Female" H 9527 2535 50  0000 L CNN
 F 2 "" H 9500 2650 50  0001 C CNN
@@
 Wire Wire Line
 	4950 3950 7100 3950
-Connection ~ 7850 5600
-Wire Wire Line
-	7850 5200 7850 5600
-Connection ~ 7850 5200
-Wire Wire Line
-	7850 4800 7850 5200
-Connection ~ 7850 4800
-Wire Wire Line
-	7850 4400 7850 4800
-Connection ~ 7850 4400
-Wire Wire Line
-	7850 3950 7850 4400
-$Comp
-L Switch:SW_SPST SW-PWR
+Wire Wire Line
+	7850 3950 7850 4350
+$Comp
+L Switch:SW_SPST SW-PWR1
 U 1 1 61C46462
 P 5000 5150
-F 0 "SW-PWR" V 4954 5248 50  0000 L CNN
+F 0 "SW-PWR1" V 4954 5248 50  0000 L CNN
 F 1 "SW_SPST" V 5045 5248 50  0000 L CNN
 F 2 "" H 5000 5150 50  0001 C CNN
@@
 Wire Wire Line
 	4550 4850 4550 4750
+Connection ~ 7850 4350
+Wire Wire Line
+	7850 4350 7850 4750
+Connection ~ 7850 4750
+Wire Wire Line
+	7850 4750 7850 5150
+Connection ~ 7850 5150
+Wire Wire Line
+	7850 5150 7850 5550
+Connection ~ 7850 5550
+Wire Wire Line
+	7850 5550 7850 5800
 $EndSCHEMATC

Commit message: improve: schematic, SW_PWR, EN
Parts:
- removed SW-PWR1: SW_SPST, symbol Switch:SW_SPST
- added SW_PWR1: SW_SPST, symbol Switch:SW_SPST
- A2: footprint ert -> blues-footprints:Notecarrier-B
Connections:
- net labels added: +BATT
- net labels removed: VCC
- wire segments 61 -> 72
- no-connect marks 19 -> 16
Other:
- note removed: "Should VIO on the Notecarrier be wired to 3.3V on the Feather?"
- note removed: "Should VUSB on the notecarrier be wired to VUSB on the Feather?"
- moved on the sheet: A1, BT-LIPO1, DBLU1, DERR1, DGRN1, DRED1, DYEL1, JDIAG1, R1, R2, R3, R4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
